Commit message: support so101 follower in gazebo

File: src/lerobot_robots_description/urdf/SO101/so101_gazebo.urdf (robot description, URDF)
Before this commit: robot so101_gazebo, 8 links, 7 joints
Links:
- removed link gripper
- added link gripperlink, mass 0.087; collision mesh filename=package://lerobot_robots_description/urdf/SO101/assets/sts3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; collision mesh filename=package://lerobot_robots_description/urdf/SO101/assets/wris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
Joints:
- removed joint J_elbow_flex
- removed joint J_gripper
- removed joint J_shoulder_lift
- removed joint J_shoulder_pan
- removed joint J_world_fixed
- removed joint J_wrist_flex
- removed joint J_wrist_roll
- added joint elbow_flex: type revolute, parent upper_arm, child lower_arm, origin xyz=-0.11257 -0.028 2.46331e-16 rpy=-1.22818e-15 5.75928e-16 1.5708, axis 0 0 1, limit lower=-1.69 upper=1.69 effort=10 velocity=10
- added joint gripper: type revolute, parent gripperlink, child moving_jaw_so101_v1, origin xyz=0.0202 0.0188 -0.0234 rpy=1.5708 -5.14108e-17 -1.38655e-14, axis 0 0 1, limit lower=-0.174533 upper=1.74533 effort=10 velocity=10
- added joint shoulder_lift: type revolute, parent shoulder, child upper_arm, origin xyz=-0.0303992 -0.0182778 -0.0542 rpy=-1.5708 -1.5708 0, axis 0 0 1, limit lower=-1.74533 upper=1.74533 effort=10 velocity=10
- added joint shoulder_pan: type revolute, parent base, child shoulder, origin xyz=0.0207909 -0.0230745 0.0948817 rpy=-3.14159 6.03684e-16 1.5708, axis 0 0 1, limit lower=-1.91986 upper=1.91986 effort=10 velocity=10
- added joint world_fixed: type fixed, parent world, child base
- added joint wrist_flex: type revolute, parent lower_arm, child wrist, origin xyz=-0.1349 0.0052 1.65232e-16 rpy=3.2474e-15 2.86219e-15 -1.5708, axis 0 0 1, limit lower=-1.65806 upper=1.65806 effort=10 velocity=10
- added joint wrist_roll: type revolute, parent wrist, child gripperlink, origin xyz=0 -0.0611 0.0181 rpy=1.5708 -9.38083e-08 3.14159, axis 0 0 1, limit lower=-2.74385 upper=2.84121 effort=10 velocity=10

Commit message: support hand camera in gazebo env

File: src/lerobot_robots_description/urdf/SO101/so101_gazebo.urdf (robot description, URDF)
Before this commit: robot so101_gazebo, 8 links, 7 joints
Links:
- added link camera_link; collision box size=0.02 0.03 0.05; visual box size=0.02 0.03 0.05
Joints:
- added joint camera_joint: type fixed, parent gripperlink, child camera_link, origin xyz=0.0 0.05 -0.03 rpy=-1.57 0.77 -1.57, axis 0 0 0
