Commit message: teleoperation started.

File: src/lerobot_robots_description/urdf/SO101/so101_new_calib.urdf (robot description, URDF)
Before this commit: robot so101_new_calib, 9 links, 8 joints
Links:
- link base: geometry collision mesh filename=package://lerobot_robots_description/urdf/SO101/assets/base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; collision mesh filename=package://lerobot_robots_description/urdf/SO101/assets/base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
- link gripper: geometry collision mesh filename=package://lerobot_robots_description/urdf/SO101/assets/sts3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; collision mesh filename=package://lerobot_robots_description/urdf/SO101/assets/wris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
- link lower_arm: geometry collision mesh filename=package://lerobot_robots_description/urdf/SO101/assets/moto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; collision mesh filename=package://lerobot_robots_description/urdf/SO101/assets/sts3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
- link moving_jaw_so101_v1: geometry collision mesh filename=package://lerobot_robots_description/urdf/SO101/assets/movi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; visual mesh filename=package://lerobot_robots_description/urdf/SO101/assets/movi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
- link shoulder: geometry collision mesh filename=package://lerobot_robots_description/urdf/SO101/assets/moto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; collision mesh filename=package://lerobot_robots_description/urdf/SO101/assets/rota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
- link upper_arm: geometry collision mesh filename=package://lerobot_robots_description/urdf/SO101/assets/sts3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; collision mesh filename=package://lerobot_robots_description/urdf/SO101/assets/uppe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
- link wrist: geometry collision mesh filename=package://lerobot_robots_description/urdf/SO101/assets/sts3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; collision mesh filename=package://lerobot_robots_description/urdf/SO101/assets/wris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

Commit message: split rewards

File: src/lerobot_robots_description/urdf/SO101/so101_new_calib.urdf (robot description, URDF)
Before this commit: robot so101_new_calib, 9 links, 8 joints
Links:
- added link ee_gripper, mass 1e-9
- added link ee_wrist, mass 1e-9
Joints:
- added joint ee_gripper_frame: type fixed, parent moving_jaw_so101_v1, child ee_gripper, origin xyz=-0.005 -0.061 0.02 rpy=1.5708 1.22465e-16 1.5708, axis 0 0 0
- added joint ee_wrist_frame: type fixed, parent wrist, child ee_wrist, origin xyz=0.012 -0.145 0.018 rpy=1.5708 1.22465e-16 1.5708, axis 0 0 0
