Commit message: forgot to disable 1 finger

File: src/lerobot_robots_description/urdf/SO101/so101_new_calib_stable_grasp.urdf (robot description, URDF)
Before this commit: robot so101_new_calib, 11 links, 10 joints
Links:
- link gripper: geometry collision box size=0.005 0.02 0.07; collision box size=0.005 0.02 0.07

Commit message: narrower inner fingers

File: src/lerobot_robots_description/urdf/SO101/so101_new_calib_stable_grasp.urdf (robot description, URDF)
Before this commit: robot so101_new_calib, 11 links, 10 joints
Links:
- link gripper: geometry collision box size=0.005 0.0175 0.07; collision box size=0.005 0.02 0.07
- link moving_jaw_so101_v1: geometry collision box size=0.005 0.07 0.0175 xyz=0 0 0.1; collision box size=0.005 0.07 0.02 xyz=0 0 0.1
